Commit message: Renaming docs folder to src.

File: mmtbot_description/urdf/table.macro.xacro (robot description, xacro)
@@ -46,5 +46,5 @@
         <!-- %%%%%%%%%%%%%%%%%%%%%%%%%%%%%%%%%%%%%%%%%%%%%-->
         <link name="${name}"/>
-        <joint name="world_to_${name}" type="fixed">
+        <joint name="${parent}_to_${name}" type="fixed">
             <parent link="${parent}"/>
             <child link="${name}" />
