Commit message: Trying to make the simulation.

File: mmtbot_description/urdf/mmtbot.urdf.xacro (robot description, xacro)
@@ -1,4 +1,4 @@
 <?xml version="1.0" ?>
-<robot name="p_moliveira" xmlns:xacro="http://ros.org/wiki/xacro">
+<robot name="mmtbot" xmlns:xacro="http://ros.org/wiki/xacro">
   <!--  Xacro description of turtlebot robot waffle pi used to play team hunt.-->
   <!--  Miguel Riem Oliveira-->
@@ -7,8 +7,9 @@
   <!--Properties are global so they can be viewed from inside the included xacros-->
   <!--  args are used with $(arg arg_name), properties are used as ${property_name}-->
-  <xacro:property name="table_height" value="0.795"/>
-  <xacro:property name="table_dimension_x" value="1.25"/>
-  <xacro:property name="table_dimension_y" value="0.9"/>
-  <xacro:property name="table_dimension_z" value="0.015"/>
+  <xacro:property name="table1_height" value="0.795"/>
+  <xacro:property name="table1_width" value="1.25"/>
+  <xacro:property name="table1_lenght" value="0.9"/>
+  <xacro:property name="table1_tabletop_thickness" value="0.015"/>
+  <xacro:property name="table1_leg_radius" value="0.02"/>
   <!-- Include other files-->
   <xacro:include filename="$(find mmtbot_description)/urdf/properties.xacro"/>
@@ -21,20 +22,30 @@
   <link name="world"/>
   <!--  Place table 1 in the scene-->
-  <xacro:table_macro table_name="table_1" parent="world" dx="${table_dimension_x}" dy="${table_dimension_y}" dz="${table_dimension_z}">
-    <origin xyz="3 0 ${table_height}" rpy="0 0 0" />
-  </xacro:table_macro>
-  <xacro:asus_camera_model name="camera_1" parent="table_1">
-    <origin xyz="0 0 0.5" rpy="0 0.3 0" />
-  </xacro:asus_camera_model>
+<!--  <xacro:table_macro name="table1" parent="world" width="${table1_width}"-->
+<!--                     lenght="${table1_lenght}" height="${table1_height}"-->
+<!--                     tabletop_thickness="${table1_tabletop_thickness}" leg_radius="${table1_leg_radius}">-->
+<!--    <origin xyz="3 0 0" rpy="0 0 0" />-->
+<!--  </xacro:table_macro>-->
+  <!--  Manipulator-->
   <xacro:ur10e_robot prefix="" joint_limited="false"/>
-  <xacro:sensor_astra parent="base_link" prefix="camera">
-      <!-- NOTE: CHANGE THIS -->
-      <origin xyz="-1 0 1" rpy="0 0 0"/>
-      <!-- <origin xyz="0.041311319304504816 -0.06402544453787727 0.044527571211305426" rpy="3.13766148064 -0.00787797070144 0.000110993634886"/> -->
-  </xacro:sensor_astra>
-  <joint name="world_joint" type="fixed">
-    <parent link="table_1" />
-    <child link = "base_link" />
-    <origin xyz="0.2 0.2 0.0" rpy="0.0 0.0 0.0" />
+  <!--  Place robot on top of the table1-->
+<!--  <joint name="tabletop_table1_to_ur10e" type="fixed">-->
+<!--    <parent link="tabletop_table1" />-->
+<!--    <child link = "base_link"/>-->
+<!--    <origin xyz="${table1_lenght/2-0.04} 0.0 0.1" rpy="0.0 0.0 0.0" />-->
+<!--  </joint>-->
+    <joint name="tabletop_table1_to_ur10e" type="fixed">
+    <parent link="world" />
+    <child link = "base_link"/>
+    <origin xyz="0 0.0 0.1" rpy="0.0 0.0 0.0" />
   </joint>
+<!--  &lt;!&ndash;  Camera 1&ndash;&gt;-->
+<!--    <xacro:asus_camera_model name="camera1" parent="ee_link">-->
+<!--      <origin xyz="0 0 0.05" rpy="0 0.3 0" />-->
+<!--    </xacro:asus_camera_model>-->
+<!--    <xacro:sensor_astra parent="base_link" prefix="camera">-->
+<!--        &lt;!&ndash; NOTE: CHANGE THIS &ndash;&gt;-->
+<!--        <origin xyz="-1 0 1" rpy="0 0 0"/>-->
+<!--        &lt;!&ndash; <origin xyz="0.041311319304504816 -0.06402544453787727 0.044527571211305426" rpy="3.13766148064 -0.00787797070144 0.000110993634886"/> &ndash;&gt;-->
+<!--    </xacro:sensor_astra>-->
 </robot>

File: mmtbot_description/urdf/table.macro.xacro (robot description, xacro)
@@ -1,40 +1,105 @@
 <?xml version="1.0"?>
 <robot name="table_macro" xmlns:xacro="http://ros.org/wiki/xacro">
-    <xacro:macro name="table_macro" params="table_name parent *origin dx dy dz">
-        <!--  <xacro:arg name="laser_visual"  default="false"/>-->
-        <!--  <xacro:arg name="camera_visual" default="false"/>-->
-        <!--  <xacro:arg name="imu_visual"    default="false"/>-->
-        <link name="${table_name}"/>
-        <link name="tabletop_${table_name}">
+    <!-- A leg macro, to be used bellow by the table macro.-->
+    <xacro:macro name="table_leg_macro" params="name parent *origin height leg_radius">
+        <link name="${parent}_${name}">
             <visual>
-                <origin xyz="${dx/2} ${dy/2} ${-dz/2}" rpy="0 0 0"/>
+                <origin xyz="0.0 0.0 ${-height/2}" rpy="0 0 0" />
                 <geometry>
-                    <box size="${dx} ${dy} ${dz}"/>
+                    <cylinder radius="${leg_radius}" length="${height}" />
+                </geometry>
+                <material name="grey"/>
+            </visual>
+            <collision>
+                <origin xyz="0.0 0.0 ${-height/2}" rpy="0 0 0" />
+                <geometry>
+                    <cylinder radius="${leg_radius}" length="${height}" />
+                </geometry>
+            </collision>
+            <inertial>
+                <mass value="1.0" />
+                <origin xyz="0.0 0.0 ${-height/2}" rpy="0 0 0" />
+                <inertia ixx="0.1" ixy="0"  ixz="0"
+                         iyy="0.1" iyz="0"
+                         izz="0.01" />
+            </inertial>
+        </link>
+        <gazebo reference="${parent}_${name}">
+            <material>Gazebo/Grey</material>
+            <mu1>1000.0</mu1>
+            <mu2>1000.0</mu2>
+            <kp>10000000.0</kp>
+            <kd>1.0</kd>
+            <selfCollide>true</selfCollide>
+        </gazebo>
+        <joint name="${parent}_to_${name}" type="fixed">
+            <parent link="${parent}" />
+            <child link="${parent}_${name}" />
+            <xacro:insert_block name="origin"/>
+        </joint>
+    </xacro:macro>
+    <!-- Table macro, the one that is called from another file.-->
+    <xacro:macro name="table_macro" params="name parent *origin width lenght height
+                                            tabletop_thickness leg_radius">
+        <!-- %%%%%%%%%%%%%%%%%%%%%%%%%%%%%%%%%%%%%%%%%%%%%-->
+        <!-- %%%%%%%%%%%%%%%%% Links %%%%%%%%%%%%%%%%%%%%%-->
+        <!-- %%%%%%%%%%%%%%%%%%%%%%%%%%%%%%%%%%%%%%%%%%%%%-->
+        <!-- table link-->
+        <link name="${name}"/>
+        <!-- tabletop link-->
+        <link name="tabletop_${name}">
+            <visual>
+                <origin xyz="0 0 ${-tabletop_thickness/2}" rpy="0 0 0"/>
+                <geometry>
+                    <box size="${width} ${lenght} ${tabletop_thickness}"/>
                 </geometry>
                 <material name="grey"/>
             </visual>
             <collision name="base_link_collision">
-                <origin xyz="${dx/2} ${dy/2} ${-dz/2}" rpy="0 0 0"/>
+                <origin xyz="0 0 ${-tabletop_thickness/2}" rpy="0 0 0"/>
                 <geometry>
-                    <box size="${dx} ${dy} ${dz}"/>
+                    <box size="${width} ${lenght} ${tabletop_thickness}"/>
                 </geometry>
             </collision>
-            <!--                <inertial>-->
-            <!--                  <origin xyz="0 0 0" rpy="0 0 0"/>-->
-            <!--                  <mass value="1.3729096e+00"/>-->
-            <!--                  <inertia ixx="8.7002718e-03" ixy="-4.7576583e-05" ixz="1.1160499e-04"-->
-            <!--                           iyy="8.6195418e-03" iyz="-3.5422299e-06"-->
-            <!--                           izz="1.4612727e-02" />-->
-            <!--                </inertial>-->
+            <inertial>
+                <mass value="1.0" />
+                <origin xyz="0 0 ${-tabletop_thickness/2}" rpy="0 0 0"/>
+                <inertia ixx="1" ixy="0"  ixz="0" iyy="1" iyz="0" izz="1" />
+            </inertial>
         </link>
-        <joint name="world_to_${table_name}" type="fixed">
+        <gazebo reference="tabletop_${name}">
+            <material>Gazebo/Grey</material>
+            <mu1>50.0</mu1>
+            <mu2>50.0</mu2>
+            <kp>1000000.0</kp>
+            <kd>1.0</kd>
+            <selfCollide>false</selfCollide>
+        </gazebo>
+        <!-- Define the four legs -->
+        <xacro:table_leg_macro name="leg1" parent="tabletop_${name}" height="${height}" leg_radius="${leg_radius}">
+            <origin xyz="${-width/2+leg_radius} ${lenght/2-leg_radius} 0" rpy="0 0 0"/>
+        </xacro:table_leg_macro>
+        <xacro:table_leg_macro name="leg2" parent="tabletop_${name}" height="${height}" leg_radius="${leg_radius}">
+            <origin xyz="${width/2-leg_radius} ${lenght/2-leg_radius} 0" rpy="0 0 0"/>
+        </xacro:table_leg_macro>
+        <xacro:table_leg_macro name="leg3" parent="tabletop_${name}" height="${height}" leg_radius="${leg_radius}">
+            <origin xyz="${width/2-leg_radius} ${-lenght/2+leg_radius} 0" rpy="0 0 0"/>
+        </xacro:table_leg_macro>
+        <xacro:table_leg_macro name="leg4" parent="tabletop_${name}" height="${height}" leg_radius="${leg_radius}">
+            <origin xyz="${-width/2+leg_radius} ${-lenght/2+leg_radius} 0" rpy="0 0 0"/>
+        </xacro:table_leg_macro>
+        <!-- %%%%%%%%%%%%%%%%%%%%%%%%%%%%%%%%%%%%%%%%%%%%%-->
+        <!-- %%%%%%%%%%%%%%%%% Joints %%%%%%%%%%%%%%%%%%%%-->
+        <!-- %%%%%%%%%%%%%%%%%%%%%%%%%%%%%%%%%%%%%%%%%%%%%-->
+        <!-- World to table1 -->
+        <joint name="world_to_${name}" type="fixed">
             <parent link="${parent}"/>
-            <child link="${table_name}" />
+            <child link="${name}" />
             <xacro:insert_block name="origin"/>
         </joint>
-        <joint name="${table_name}_to_tabletop_${table_name}" type="fixed">
-            <parent link="${table_name}"/>
-            <child link="tabletop_${table_name}" />
-            <origin xyz="0 0 0" rpy="0 0 0"/>
+        <joint name="${name}_to_tabletop_${name}" type="fixed">
+            <parent link="${name}"/>
+            <child link="tabletop_${name}" />
+            <origin xyz="0 0 ${height}" rpy="0 0 0"/>
         </joint>
     </xacro:macro>

Commit message: https://github.com/lardemua/atom/issues/241
working of the mmbot

File: mmtbot_description/urdf/mmtbot.urdf.xacro (robot description, xacro)
@@ -1,51 +1,58 @@
 <?xml version="1.0" ?>
 <robot name="mmtbot" xmlns:xacro="http://ros.org/wiki/xacro">
-  <!--  Xacro description of turtlebot robot waffle pi used to play team hunt.-->
-  <!--  Miguel Riem Oliveira-->
-  <!--  PARI, November 2020-->
-  <!--Args are local, properties are global, so we copy the values of the arguments to the properties-->
-  <!--Properties are global so they can be viewed from inside the included xacros-->
-  <!--  args are used with $(arg arg_name), properties are used as ${property_name}-->
-  <xacro:property name="table1_height" value="0.795"/>
-  <xacro:property name="table1_width" value="1.25"/>
-  <xacro:property name="table1_lenght" value="0.9"/>
-  <xacro:property name="table1_tabletop_thickness" value="0.015"/>
-  <xacro:property name="table1_leg_radius" value="0.02"/>
-  <!-- Include other files-->
-  <xacro:include filename="$(find mmtbot_description)/urdf/properties.xacro"/>
-  <xacro:include filename="$(find mmtbot_description)/urdf/table.macro.xacro"/>
-  <xacro:include filename="$(find hector_sensors_description)/urdf/asus_camera.urdf.xacro"/>
-  <xacro:include filename="$(find ur_e_description)/urdf/astra.urdf.xacro" />
-  <xacro:include filename="$(find ur_e_description)/urdf/common.gazebo.xacro" />
-  <xacro:include filename="$(find ur_e_description)/urdf/ur10e.urdf.xacro" />
-  <!-- Links and joints-->
-  <link name="world"/>
-  <!--  Place table 1 in the scene-->
-<!--  <xacro:table_macro name="table1" parent="world" width="${table1_width}"-->
-<!--                     lenght="${table1_lenght}" height="${table1_height}"-->
-<!--                     tabletop_thickness="${table1_tabletop_thickness}" leg_radius="${table1_leg_radius}">-->
-<!--    <origin xyz="3 0 0" rpy="0 0 0" />-->
-<!--  </xacro:table_macro>-->
-  <!--  Manipulator-->
-  <xacro:ur10e_robot prefix="" joint_limited="false"/>
-  <!--  Place robot on top of the table1-->
-<!--  <joint name="tabletop_table1_to_ur10e" type="fixed">-->
-<!--    <parent link="tabletop_table1" />-->
-<!--    <child link = "base_link"/>-->
-<!--    <origin xyz="${table1_lenght/2-0.04} 0.0 0.1" rpy="0.0 0.0 0.0" />-->
-<!--  </joint>-->
+    <!--  Xacro description of turtlebot robot waffle pi used to play team hunt.-->
+    <!--  Miguel Riem Oliveira-->
+    <!--  PARI, November 2020-->
+    <!--Args are local, properties are global, so we copy the values of the arguments to the properties-->
+    <!--Properties are global so they can be viewed from inside the included xacros-->
+    <!--  args are used with $(arg arg_name), properties are used as ${property_name}-->
+    <xacro:property name="table1_height" value="0.795"/>
+    <xacro:property name="table1_width" value=".9"/>
+    <xacro:property name="table1_lenght" value="0.9"/>
+    <xacro:property name="table1_tabletop_thickness" value="0.015"/>
+    <xacro:property name="table1_leg_radius" value="0.02"/>
+    <xacro:property name="pi" value="3.1415"/>
+    <!-- Include other files-->
+    <xacro:include filename="$(find mmtbot_description)/urdf/properties.xacro"/>
+    <xacro:include filename="$(find mmtbot_description)/urdf/table.macro.xacro"/>
+    <xacro:include filename="$(find mmtbot_description)/urdf/tripod.macro.xacro"/>
+    <xacro:include filename="$(find hector_sensors_description)/urdf/asus_camera.urdf.xacro"/>
+    <xacro:include filename="$(find hector_sensors_description)/urdf/vlp16.urdf.xacro"/>
+    <xacro:include filename="$(find ur_e_description)/urdf/astra.urdf.xacro" />
+    <xacro:include filename="$(find ur_e_description)/urdf/common.gazebo.xacro" />
+    <xacro:include filename="$(find ur_e_description)/urdf/ur10e.urdf.xacro" />
+    <xacro:include filename="$(find hector_xacro_tools)/urdf/inertia_tensors.urdf.xacro"/>
+    <!-- Links and joints-->
+    <link name="world"/>
+    <!-- Place table 1 in the scene-->
+    <xacro:table_macro name="table1" parent="world" width="${table1_width}"
+                       lenght="${table1_lenght}" height="${table1_height}"
+                       tabletop_thickness="${table1_tabletop_thickness}" leg_radius="${table1_leg_radius}">
+        <origin xyz="1.5 0 0" rpy="0 0 ${pi/2}" />
+    </xacro:table_macro>
+    <!--  Manipulator-->
+    <xacro:ur10e_robot prefix="" joint_limited="false"/>
+    <!--  Place robot on top of the table1-->
     <joint name="tabletop_table1_to_ur10e" type="fixed">
-    <parent link="world" />
-    <child link = "base_link"/>
-    <origin xyz="0 0.0 0.1" rpy="0.0 0.0 0.0" />
-  </joint>
-<!--  &lt;!&ndash;  Camera 1&ndash;&gt;-->
-<!--    <xacro:asus_camera_model name="camera1" parent="ee_link">-->
-<!--      <origin xyz="0 0 0.05" rpy="0 0.3 0" />-->
-<!--    </xacro:asus_camera_model>-->
-<!--    <xacro:sensor_astra parent="base_link" prefix="camera">-->
-<!--        &lt;!&ndash; NOTE: CHANGE THIS &ndash;&gt;-->
-<!--        <origin xyz="-1 0 1" rpy="0 0 0"/>-->
-<!--        &lt;!&ndash; <origin xyz="0.041311319304504816 -0.06402544453787727 0.044527571211305426" rpy="3.13766148064 -0.00787797070144 0.000110993634886"/> &ndash;&gt;-->
-<!--    </xacro:sensor_astra>-->
+        <parent link="tabletop_table1" />
+        <child link = "base_link"/>
+        <origin xyz="0.0 0.0 0.001" rpy="0.0 0.0 0.0" />
+    </joint>
+    <!-- Hand eye camera-->
+    <xacro:asus_camera_model name="camera1" parent="ee_link">
+        <origin xyz="0 0 0.06" rpy="0 0.3 0" />
+    </xacro:asus_camera_model>
+    <!--  <xacro:sensor_astra parent="base_link" prefix="camera">-->
+    <!--    &lt;!&ndash; NOTE: CHANGE THIS &ndash;&gt;-->
+    <!--    <origin xyz="-1 0 1" rpy="0 0 0"/>-->
+    <!--    &lt;!&ndash; <origin xyz="0.041311319304504816 -0.06402544453787727 0.044527571211305426" rpy="3.13766148064 -0.00787797070144 0.000110993634886"/> &ndash;&gt;-->
+    <!--  </xacro:sensor_astra>-->
+    <!-- Place tripod1 in the scene-->
+    <xacro:tripod_macro name="tripod1" parent="world">
+        <origin xyz="-0.5 0 0" rpy="0 0 ${pi/3}" />
+    </xacro:tripod_macro>
+    <!-- Velodyne Support-->
+    <xacro:vlp16_model name="3dlidar" parent="tripod1_plate">
+        <origin xyz="0 0 0.04" rpy="0 ${pi/10} 0" />
+    </xacro:vlp16_model>
 </robot>

File: mmtbot_description/urdf/table.macro.xacro (robot description, xacro)
@@ -5,5 +5,5 @@
         <link name="${parent}_${name}">
             <visual>
-                <origin xyz="0.0 0.0 ${-height/2}" rpy="0 0 0" />
+                <origin xyz="0.0 0.0 ${height/2}" rpy="0 0 0" />
                 <geometry>
                     <cylinder radius="${leg_radius}" length="${height}" />
@@ -12,5 +12,5 @@
             </visual>
             <collision>
-                <origin xyz="0.0 0.0 ${-height/2}" rpy="0 0 0" />
+                <origin xyz="0.0 0.0 ${height/2}" rpy="0 0 0" />
                 <geometry>
                     <cylinder radius="${leg_radius}" length="${height}" />
@@ -19,5 +19,5 @@
             <inertial>
                 <mass value="1.0" />
-                <origin xyz="0.0 0.0 ${-height/2}" rpy="0 0 0" />
+                <origin xyz="0.0 0.0 ${height/2}" rpy="0 0 0" />
                 <inertia ixx="0.1" ixy="0"  ixz="0"
                          iyy="0.1" iyz="0"
@@ -43,9 +43,15 @@
                                             tabletop_thickness leg_radius">
         <!-- %%%%%%%%%%%%%%%%%%%%%%%%%%%%%%%%%%%%%%%%%%%%%-->
-        <!-- %%%%%%%%%%%%%%%%% Links %%%%%%%%%%%%%%%%%%%%%-->
+        <!-- table link-->
         <!-- %%%%%%%%%%%%%%%%%%%%%%%%%%%%%%%%%%%%%%%%%%%%%-->
-        <!-- table link-->
         <link name="${name}"/>
+        <joint name="world_to_${name}" type="fixed">
+            <parent link="${parent}"/>
+            <child link="${name}" />
+            <xacro:insert_block name="origin"/>
+        </joint>
+        <!-- %%%%%%%%%%%%%%%%%%%%%%%%%%%%%%%%%%%%%%%%%%%%%-->
         <!-- tabletop link-->
+        <!-- %%%%%%%%%%%%%%%%%%%%%%%%%%%%%%%%%%%%%%%%%%%%%-->
         <link name="tabletop_${name}">
             <visual>
@@ -76,31 +82,24 @@
             <selfCollide>false</selfCollide>
         </gazebo>
-        <!-- Define the four legs -->
-        <xacro:table_leg_macro name="leg1" parent="tabletop_${name}" height="${height}" leg_radius="${leg_radius}">
-            <origin xyz="${-width/2+leg_radius} ${lenght/2-leg_radius} 0" rpy="0 0 0"/>
-        </xacro:table_leg_macro>
-        <xacro:table_leg_macro name="leg2" parent="tabletop_${name}" height="${height}" leg_radius="${leg_radius}">
-            <origin xyz="${width/2-leg_radius} ${lenght/2-leg_radius} 0" rpy="0 0 0"/>
-        </xacro:table_leg_macro>
-        <xacro:table_leg_macro name="leg3" parent="tabletop_${name}" height="${height}" leg_radius="${leg_radius}">
-            <origin xyz="${width/2-leg_radius} ${-lenght/2+leg_radius} 0" rpy="0 0 0"/>
-        </xacro:table_leg_macro>
-        <xacro:table_leg_macro name="leg4" parent="tabletop_${name}" height="${height}" leg_radius="${leg_radius}">
-            <origin xyz="${-width/2+leg_radius} ${-lenght/2+leg_radius} 0" rpy="0 0 0"/>
-        </xacro:table_leg_macro>
-        <!-- %%%%%%%%%%%%%%%%%%%%%%%%%%%%%%%%%%%%%%%%%%%%%-->
-        <!-- %%%%%%%%%%%%%%%%% Joints %%%%%%%%%%%%%%%%%%%%-->
-        <!-- %%%%%%%%%%%%%%%%%%%%%%%%%%%%%%%%%%%%%%%%%%%%%-->
-        <!-- World to table1 -->
-        <joint name="world_to_${name}" type="fixed">
-            <parent link="${parent}"/>
-            <child link="${name}" />
-            <xacro:insert_block name="origin"/>
-        </joint>
-        <joint name="${name}_to_tabletop_${name}" type="fixed">
+         <joint name="${name}_to_tabletop_${name}" type="fixed">
             <parent link="${name}"/>
             <child link="tabletop_${name}" />
             <origin xyz="0 0 ${height}" rpy="0 0 0"/>
         </joint>
+        <!-- %%%%%%%%%%%%%%%%%%%%%%%%%%%%%%%%%%%%%%%%%%%%%-->
+        <!-- Define the four legs -->
+        <!-- %%%%%%%%%%%%%%%%%%%%%%%%%%%%%%%%%%%%%%%%%%%%%-->
+        <xacro:table_leg_macro name="leg1" parent="${name}" height="${height}" leg_radius="${leg_radius}">
+            <origin xyz="${-width/2+leg_radius} ${lenght/2-leg_radius} 0" rpy="0 0 0"/>
+        </xacro:table_leg_macro>
+        <xacro:table_leg_macro name="leg2" parent="${name}" height="${height}" leg_radius="${leg_radius}">
+            <origin xyz="${width/2-leg_radius} ${lenght/2-leg_radius} 0" rpy="0 0 0"/>
+        </xacro:table_leg_macro>
+        <xacro:table_leg_macro name="leg3" parent="${name}" height="${height}" leg_radius="${leg_radius}">
+            <origin xyz="${width/2-leg_radius} ${-lenght/2+leg_radius} 0" rpy="0 0 0"/>
+        </xacro:table_leg_macro>
+        <xacro:table_leg_macro name="leg4" parent="${name}" height="${height}" leg_radius="${leg_radius}">
+            <origin xyz="${-width/2+leg_radius} ${-lenght/2+leg_radius} 0" rpy="0 0 0"/>
+        </xacro:table_leg_macro>
     </xacro:macro>
 </robot>

Commit message: lardemua/atom#241 Puttin the objects in the propper place.

File: mmtbot_description/urdf/mmtbot.urdf.xacro (robot description, xacro)
@@ -29,5 +29,5 @@
                        lenght="${table1_lenght}" height="${table1_height}"
                        tabletop_thickness="${table1_tabletop_thickness}" leg_radius="${table1_leg_radius}">
-        <origin xyz="1.5 0 0" rpy="0 0 ${pi/2}" />
+        <origin xyz="-1 0 0" rpy="0 0 ${pi/2}" />
     </xacro:table_macro>
     <!--  Manipulator-->
@@ -40,7 +40,10 @@
     </joint>
     <!-- Hand eye camera-->
-    <xacro:asus_camera_model name="camera1" parent="ee_link">
-        <origin xyz="0 0 0.06" rpy="0 0.3 0" />
-    </xacro:asus_camera_model>
+<!--    <xacro:asus_camera_model name="camera1" parent="ee_link">-->
+<!--        <origin xyz="0 0 0.06" rpy="0 0.3 0" />-->
+<!--    </xacro:asus_camera_model>-->
+    <xacro:sensor_astra prefix="camera1" parent="ee_link">
+        <origin xyz="-0.02 0.05 0.07" rpy="0 0.2 0" />
+    </xacro:sensor_astra>
     <!--  <xacro:sensor_astra parent="base_link" prefix="camera">-->
     <!--    &lt;!&ndash; NOTE: CHANGE THIS &ndash;&gt;-->
@@ -50,5 +53,5 @@
     <!-- Place tripod1 in the scene-->
     <xacro:tripod_macro name="tripod1" parent="world">
-        <origin xyz="-0.5 0 0" rpy="0 0 ${pi/3}" />
+        <origin xyz="1 0 0" rpy="0 0 ${2/3*pi}" />
     </xacro:tripod_macro>
     <!-- Velodyne Support-->
