Commit message: lardemua/atom#241 Added charuco simulation model.

File: mmtbot_description/urdf/mmtbot.urdf.xacro (robot description, xacro)
@@ -1,7 +1,6 @@
 <?xml version="1.0" ?>
 <robot name="mmtbot" xmlns:xacro="http://ros.org/wiki/xacro">
-    <!--  Xacro description of turtlebot robot waffle pi used to play team hunt.-->
     <!--  Miguel Riem Oliveira-->
-    <!--  PARI, November 2020-->
+    <!--  February 2021-->
     <!--Args are local, properties are global, so we copy the values of the arguments to the properties-->
     <!--Properties are global so they can be viewed from inside the included xacros-->
@@ -12,15 +11,15 @@
     <xacro:property name="table1_tabletop_thickness" value="0.015"/>
     <xacro:property name="table1_leg_radius" value="0.02"/>
-    <xacro:property name="pi" value="3.1415"/>
+    <xacro:property name="M_PI" value="3.1415926535897931" />
     <!-- Include other files-->
     <xacro:include filename="$(find mmtbot_description)/urdf/properties.xacro"/>
     <xacro:include filename="$(find mmtbot_description)/urdf/table.macro.xacro"/>
     <xacro:include filename="$(find mmtbot_description)/urdf/tripod.macro.xacro"/>
-    <xacro:include filename="$(find hector_sensors_description)/urdf/asus_camera.urdf.xacro"/>
-    <xacro:include filename="$(find hector_sensors_description)/urdf/vlp16.urdf.xacro"/>
+<!--    <xacro:include filename="$(find hector_sensors_description)/urdf/asus_camera.urdf.xacro"/>-->
+<!--    <xacro:include filename="$(find hector_sensors_description)/urdf/vlp16.urdf.xacro"/>-->
     <xacro:include filename="$(find ur_e_description)/urdf/astra.urdf.xacro" />
     <xacro:include filename="$(find ur_e_description)/urdf/common.gazebo.xacro" />
     <xacro:include filename="$(find ur_e_description)/urdf/ur10e.urdf.xacro" />
-    <xacro:include filename="$(find hector_xacro_tools)/urdf/inertia_tensors.urdf.xacro"/>
+    <xacro:include filename="$(find velodyne_description)/urdf/VLP-16.urdf.xacro"/>
     <!-- Links and joints-->
     <link name="world"/>
@@ -29,5 +28,5 @@
                        lenght="${table1_lenght}" height="${table1_height}"
                        tabletop_thickness="${table1_tabletop_thickness}" leg_radius="${table1_leg_radius}">
-        <origin xyz="-1 0 0" rpy="0 0 ${pi/2}" />
+        <origin xyz="-1 0 0" rpy="0 0 ${M_PI/2}" />
     </xacro:table_macro>
     <!--  Manipulator-->
@@ -39,8 +38,4 @@
         <origin xyz="0.0 0.0 0.001" rpy="0.0 0.0 0.0" />
     </joint>
-    <!-- Hand eye camera-->
-<!--    <xacro:asus_camera_model name="camera1" parent="ee_link">-->
-<!--        <origin xyz="0 0 0.06" rpy="0 0.3 0" />-->
-<!--    </xacro:asus_camera_model>-->
     <xacro:sensor_astra prefix="camera1" parent="ee_link">
         <origin xyz="-0.02 0.05 0.07" rpy="0 0.2 0" />
@@ -53,9 +48,9 @@
     <!-- Place tripod1 in the scene-->
     <xacro:tripod_macro name="tripod1" parent="world">
-        <origin xyz="1 0 0" rpy="0 0 ${2/3*pi}" />
+        <origin xyz="1 0 0" rpy="0 0 ${2/3*M_PI}" />
     </xacro:tripod_macro>
-    <!-- Velodyne Support-->
-    <xacro:vlp16_model name="3dlidar" parent="tripod1_plate">
-        <origin xyz="0 0 0.04" rpy="0 ${pi/10} 0" />
-    </xacro:vlp16_model>
+    <!-- Put 3d lidar in the scene-->
+    <xacro:VLP-16 name="3dlidar" parent="tripod1_plate">
+        <origin xyz="0 0 0.04" rpy="0 ${M_PI/10} 0" />
+    </xacro:VLP-16>
 </robot>

Commit message: lardemua/atom#241 I have extended the scenario to include a second astra camera. That way, using only lidar and rgb we have 3 sensors.

File: mmtbot_description/urdf/mmtbot.urdf.xacro (robot description, xacro)
@@ -38,5 +38,5 @@
         <origin xyz="0.0 0.0 0.001" rpy="0.0 0.0 0.0" />
     </joint>
-    <xacro:sensor_astra prefix="camera1" parent="ee_link">
+    <xacro:sensor_astra prefix="hand_camera" parent="ee_link">
         <origin xyz="-0.02 0.05 0.07" rpy="0 0.2 0" />
     </xacro:sensor_astra>
@@ -51,6 +51,9 @@
     </xacro:tripod_macro>
     <!-- Put 3d lidar in the scene-->
-    <xacro:VLP-16 name="3dlidar" parent="tripod1_plate">
-        <origin xyz="0 0 0.04" rpy="0 ${M_PI/10} 0" />
+    <xacro:VLP-16 name="lidar" parent="tripod1_left_support">
+        <origin xyz="0 0 0.001" rpy="0 0 0" />
     </xacro:VLP-16>
+    <xacro:sensor_astra prefix="world_camera" parent="tripod1_right_support">
+        <origin xyz="0.02 0.07 0.015" rpy="0 0.0 0" />
+    </xacro:sensor_astra>
 </robot>

File: mmtbot_description/urdf/tripod.macro.xacro (robot description, xacro)
@@ -38,10 +38,61 @@
         <xacro:insert_block name="origin"/>
     </joint>
-    <link name="${name}_plate"/>
+    <gazebo reference="${name}">
+        <material>Gazebo/Grey</material>
+        <mu1>50.0</mu1>
+        <mu2>50.0</mu2>
+        <kp>1000000.0</kp>
+        <kd>1.0</kd>
+        <selfCollide>false</selfCollide>
+    </gazebo>
+    <link name="${name}_plate">
+        <visual>
+            <origin xyz="0 0 0" rpy="0 0 0"/>
+            <geometry>
+                <box size="0.04 0.4 0.015"/>
+            </geometry>
+            <material name="grey"/>
+        </visual>
+        <collision name="tripod_collision">
+            <origin xyz="0 0 0" rpy="0 0 0"/>
+            <geometry>
+                <box size="0.04 0.15 0.015"/>
+            </geometry>
+        </collision>
+        <inertial>
+            <mass value="1.0" />
+            <origin xyz="0 0 0" rpy="0 0 0"/>
+            <inertia ixx="1" ixy="0"  ixz="0" iyy="1" iyz="0" izz="1" />
+        </inertial>
+    </link>
+    <gazebo reference="${name}">
+        <material>Gazebo/Grey</material>
+        <mu1>50.0</mu1>
+        <mu2>50.0</mu2>
+        <kp>1000000.0</kp>
+        <kd>1.0</kd>
+        <selfCollide>false</selfCollide>
+    </gazebo>
     <!-- tripod to tripod plate-->
     <joint name="${name}_to_${name}_plate" type="fixed">
         <parent link="${name}"/>
         <child link="${name}_plate" />
-        <origin xyz=".01 .03 1.32" rpy="0 0 0"/>
+        <origin xyz=".01 .03 1.32" rpy="0 ${M_PI/10} 0"/>
+    </joint>
+    <!-- Tripod left support-->
+    <link name="${name}_left_support"/>
+    <!-- tripod plate to tripod left support -->
+    <joint name="${name}_plate_to_${name}_left_support" type="fixed">
+        <parent link="${name}_plate"/>
+        <child link="${name}_left_support" />
+        <origin xyz="0 0.18 0.0075" rpy="0 0 0"/>
+    </joint>
+    <!-- Tripod right support-->
+    <link name="${name}_right_support"/>
+    <!-- tripod plate to tripod right support -->
+    <joint name="${name}_plate_to_${name}_right_support" type="fixed">
+        <parent link="${name}_plate"/>
+        <child link="${name}_right_support" />
+        <origin xyz="0 -0.18 0.0075" rpy="0 0 0"/>
     </joint>
     </xacro:macro>

Commit message: lardemua/atom#241 Adding record.launch

File: mmtbot_description/urdf/mmtbot.urdf.xacro (robot description, xacro)
@@ -39,5 +39,5 @@
     </joint>
     <xacro:sensor_astra prefix="hand_camera" parent="ee_link">
-        <origin xyz="-0.02 0.05 0.07" rpy="0 0.2 0" />
+        <origin xyz="-0.02 0.05 0.07" rpy="0 0.0 0" />
     </xacro:sensor_astra>
     <!--  <xacro:sensor_astra parent="base_link" prefix="camera">-->

Commit message: lardemua/atom#241 Renaming a couple of frames ...

File: mmtbot_description/urdf/mmtbot.urdf.xacro (robot description, xacro)
@@ -6,9 +6,9 @@
     <!--Properties are global so they can be viewed from inside the included xacros-->
     <!--  args are used with $(arg arg_name), properties are used as ${property_name}-->
-    <xacro:property name="table1_height" value="0.795"/>
-    <xacro:property name="table1_width" value=".9"/>
-    <xacro:property name="table1_lenght" value="0.9"/>
-    <xacro:property name="table1_tabletop_thickness" value="0.015"/>
-    <xacro:property name="table1_leg_radius" value="0.02"/>
+    <xacro:property name="table_height" value="0.795"/>
+    <xacro:property name="table_width" value=".9"/>
+    <xacro:property name="table_lenght" value="0.9"/>
+    <xacro:property name="table_tabletop_thickness" value="0.015"/>
+    <xacro:property name="table_leg_radius" value="0.02"/>
     <xacro:property name="M_PI" value="3.1415926535897931" />
     <!-- Include other files-->
@@ -16,6 +16,4 @@
     <xacro:include filename="$(find mmtbot_description)/urdf/table.macro.xacro"/>
     <xacro:include filename="$(find mmtbot_description)/urdf/tripod.macro.xacro"/>
-<!--    <xacro:include filename="$(find hector_sensors_description)/urdf/asus_camera.urdf.xacro"/>-->
-<!--    <xacro:include filename="$(find hector_sensors_description)/urdf/vlp16.urdf.xacro"/>-->
     <xacro:include filename="$(find ur_e_description)/urdf/astra.urdf.xacro" />
     <xacro:include filename="$(find ur_e_description)/urdf/common.gazebo.xacro" />
@@ -25,7 +23,7 @@
     <link name="world"/>
     <!-- Place table 1 in the scene-->
-    <xacro:table_macro name="table1" parent="world" width="${table1_width}"
-                       lenght="${table1_lenght}" height="${table1_height}"
-                       tabletop_thickness="${table1_tabletop_thickness}" leg_radius="${table1_leg_radius}">
+    <xacro:table_macro name="table" parent="world" width="${table_width}"
+                       lenght="${table_lenght}" height="${table_height}"
+                       tabletop_thickness="${table_tabletop_thickness}" leg_radius="${table_leg_radius}">
         <origin xyz="-1 0 0" rpy="0 0 ${M_PI/2}" />
     </xacro:table_macro>
@@ -33,6 +31,6 @@
     <xacro:ur10e_robot prefix="" joint_limited="false"/>
     <!--  Place robot on top of the table1-->
-    <joint name="tabletop_table1_to_ur10e" type="fixed">
-        <parent link="tabletop_table1" />
+    <joint name="tabletop_table_to_ur10e" type="fixed">
+        <parent link="tabletop_table" />
         <child link = "base_link"/>
         <origin xyz="0.0 0.0 0.001" rpy="0.0 0.0 0.0" />
@@ -41,18 +39,13 @@
         <origin xyz="-0.02 0.05 0.07" rpy="0 0.0 0" />
     </xacro:sensor_astra>
-    <!--  <xacro:sensor_astra parent="base_link" prefix="camera">-->
-    <!--    &lt;!&ndash; NOTE: CHANGE THIS &ndash;&gt;-->
-    <!--    <origin xyz="-1 0 1" rpy="0 0 0"/>-->
-    <!--    &lt;!&ndash; <origin xyz="0.041311319304504816 -0.06402544453787727 0.044527571211305426" rpy="3.13766148064 -0.00787797070144 0.000110993634886"/> &ndash;&gt;-->
-    <!--  </xacro:sensor_astra>-->
-    <!-- Place tripod1 in the scene-->
-    <xacro:tripod_macro name="tripod1" parent="world">
+    <!-- Place tripod in the scene-->
+    <xacro:tripod_macro name="tripod" parent="world">
         <origin xyz="1 0 0" rpy="0 0 ${2/3*M_PI}" />
     </xacro:tripod_macro>
     <!-- Put 3d lidar in the scene-->
-    <xacro:VLP-16 name="lidar" parent="tripod1_left_support">
+    <xacro:VLP-16 name="3dlidar" parent="tripod_left_support" >
         <origin xyz="0 0 0.001" rpy="0 0 0" />
     </xacro:VLP-16>
-    <xacro:sensor_astra prefix="world_camera" parent="tripod1_right_support">
+    <xacro:sensor_astra prefix="world_camera" parent="tripod_right_support">
         <origin xyz="0.02 0.07 0.015" rpy="0 0.0 0" />
     </xacro:sensor_astra>

File: mmtbot_description/urdf/table.macro.xacro (robot description, xacro)
@@ -2,10 +2,10 @@
 <robot name="table_macro" xmlns:xacro="http://ros.org/wiki/xacro">
     <!-- A leg macro, to be used bellow by the table macro.-->
-    <xacro:macro name="table_leg_macro" params="name parent *origin height leg_radius">
-        <link name="${parent}_${name}">
+    <xacro:macro name="table_leg_macro" params="name parent *origin height leg_radius tabletop_thickness">
+        <link name="${name}_${parent}">
             <visual>
-                <origin xyz="0.0 0.0 ${height/2}" rpy="0 0 0" />
+                <origin xyz="0.0 0.0 ${height/2-tabletop_thickness}" rpy="0 0 0" />
                 <geometry>
-                    <cylinder radius="${leg_radius}" length="${height}" />
+                    <cylinder radius="${leg_radius}" length="${height-tabletop_thickness}" />
                 </geometry>
                 <material name="grey"/>
@@ -14,10 +14,10 @@
                 <origin xyz="0.0 0.0 ${height/2}" rpy="0 0 0" />
                 <geometry>
-                    <cylinder radius="${leg_radius}" length="${height}" />
+                    <cylinder radius="${leg_radius}" length="${height-tabletop_thickness}" />
                 </geometry>
             </collision>
             <inertial>
                 <mass value="1.0" />
-                <origin xyz="0.0 0.0 ${height/2}" rpy="0 0 0" />
+                <origin xyz="0.0 0.0 ${height/2-tabletop_thickness}" rpy="0 0 0" />
                 <inertia ixx="0.1" ixy="0"  ixz="0"
                          iyy="0.1" iyz="0"
@@ -25,5 +25,5 @@
             </inertial>
         </link>
-        <gazebo reference="${parent}_${name}">
+        <gazebo reference="${name}_${parent}">
             <material>Gazebo/Grey</material>
             <mu1>1000.0</mu1>
@@ -35,5 +35,5 @@
         <joint name="${parent}_to_${name}" type="fixed">
             <parent link="${parent}" />
-            <child link="${parent}_${name}" />
+            <child link="${name}_${parent}" />
             <xacro:insert_block name="origin"/>
         </joint>
@@ -56,5 +56,5 @@
         <link name="tabletop_${name}">
             <visual>
-                <origin xyz="0 0 ${-tabletop_thickness/2}" rpy="0 0 0"/>
+                <origin xyz="0 0 ${-tabletop_thickness}" rpy="0 0 0"/>
                 <geometry>
                     <box size="${width} ${lenght} ${tabletop_thickness}"/>
@@ -63,5 +63,5 @@
             </visual>
             <collision name="base_link_collision">
-                <origin xyz="0 0 ${-tabletop_thickness/2}" rpy="0 0 0"/>
+                <origin xyz="0 0 ${-tabletop_thickness}" rpy="0 0 0"/>
                 <geometry>
                     <box size="${width} ${lenght} ${tabletop_thickness}"/>
@@ -70,5 +70,5 @@
             <inertial>
                 <mass value="1.0" />
-                <origin xyz="0 0 ${-tabletop_thickness/2}" rpy="0 0 0"/>
+                <origin xyz="0 0 ${-tabletop_thickness}" rpy="0 0 0"/>
                 <inertia ixx="1" ixy="0"  ixz="0" iyy="1" iyz="0" izz="1" />
             </inertial>
@@ -90,14 +90,14 @@
         <!-- Define the four legs -->
         <!-- %%%%%%%%%%%%%%%%%%%%%%%%%%%%%%%%%%%%%%%%%%%%%-->
-        <xacro:table_leg_macro name="leg1" parent="${name}" height="${height}" leg_radius="${leg_radius}">
+        <xacro:table_leg_macro name="leg1" parent="${name}" height="${height}" leg_radius="${leg_radius}" tabletop_thickness="${tabletop_thickness}">
             <origin xyz="${-width/2+leg_radius} ${lenght/2-leg_radius} 0" rpy="0 0 0"/>
         </xacro:table_leg_macro>
-        <xacro:table_leg_macro name="leg2" parent="${name}" height="${height}" leg_radius="${leg_radius}">
+        <xacro:table_leg_macro name="leg2" parent="${name}" height="${height}" leg_radius="${leg_radius}" tabletop_thickness="${tabletop_thickness}">
             <origin xyz="${width/2-leg_radius} ${lenght/2-leg_radius} 0" rpy="0 0 0"/>
         </xacro:table_leg_macro>
-        <xacro:table_leg_macro name="leg3" parent="${name}" height="${height}" leg_radius="${leg_radius}">
+        <xacro:table_leg_macro name="leg3" parent="${name}" height="${height}" leg_radius="${leg_radius}" tabletop_thickness="${tabletop_thickness}">
             <origin xyz="${width/2-leg_radius} ${-lenght/2+leg_radius} 0" rpy="0 0 0"/>
         </xacro:table_leg_macro>
-        <xacro:table_leg_macro name="leg4" parent="${name}" height="${height}" leg_radius="${leg_radius}">
+        <xacro:table_leg_macro name="leg4" parent="${name}" height="${height}" leg_radius="${leg_radius}" tabletop_thickness="${tabletop_thickness}">
             <origin xyz="${-width/2+leg_radius} ${-lenght/2+leg_radius} 0" rpy="0 0 0"/>
         </xacro:table_leg_macro>

File: mmtbot_description/urdf/tripod.macro.xacro (robot description, xacro)
@@ -78,5 +78,5 @@
         <parent link="${name}"/>
         <child link="${name}_plate" />
-        <origin xyz=".01 .03 1.32" rpy="0 ${M_PI/10} 0"/>
+        <origin xyz=".01 .03 1.33" rpy="0 ${M_PI/10} 0"/>
     </joint>
     <!-- Tripod left support-->

Commit message: trying to run simulation with 3lidars to create interactive markers to align frames on rviz

File: mmtbot_description/urdf/mmtbot.urdf.xacro (robot description, xacro)
@@ -44,6 +44,12 @@
     </xacro:tripod_macro>
     <!-- Put 3d lidar in the scene-->
-    <xacro:VLP-16 name="3dlidar" parent="tripod_left_support" topic="/3dlidar/points">
+    <xacro:VLP-16 name="3dlidar_1" parent="tripod_left_support" topic="/3dlidar_1/points">
         <origin xyz="0 0 0.001" rpy="0 0 0" />
+    </xacro:VLP-16>
+    <xacro:VLP-16 name="3dlidar_2" parent="tripod_left_support" topic="/3dlidar_2/points">
+        <origin xyz="0.5 0 0.001" rpy="0 0 0" />
+    </xacro:VLP-16>
+    <xacro:VLP-16 name="3dlidar_3" parent="tripod_left_support" topic="/3dlidar_3/points">
+        <origin xyz="1 0 0.001" rpy="0 0 0" />
     </xacro:VLP-16>
     <xacro:sensor_astra prefix="world_camera" parent="tripod_right_support">

Commit message: Fixes lardemua/larcc#17

File: mmtbot_description/urdf/mmtbot.urdf.xacro (robot description, xacro)
@@ -1,9 +1,12 @@
 <?xml version="1.0" ?>
 <robot name="mmtbot" xmlns:xacro="http://ros.org/wiki/xacro">
-    <!--  Miguel Riem Oliveira-->
-    <!--  February 2021-->
+    <!-- ####################################### -->
+    <!-- Arguments and propperties-->
+    <!-- ####################################### -->
     <!--Args are local, properties are global, so we copy the values of the arguments to the properties-->
     <!--Properties are global so they can be viewed from inside the included xacros-->
     <!--  args are used with $(arg arg_name), properties are used as ${property_name}-->
+    <xacro:property name="M_PI" value="3.1415926535897931" />
+    <!-- Tables properties-->
     <xacro:property name="table_height" value="0.795"/>
     <xacro:property name="table_width" value=".9"/>
@@ -11,24 +14,5 @@
     <xacro:property name="table_tabletop_thickness" value="0.015"/>
     <xacro:property name="table_leg_radius" value="0.02"/>
-    <xacro:property name="M_PI" value="3.1415926535897931" />
-    <!-- Include other files-->
-    <xacro:include filename="$(find mmtbot_description)/urdf/properties.xacro"/>
-    <xacro:include filename="$(find mmtbot_description)/urdf/table.macro.xacro"/>
-    <xacro:include filename="$(find mmtbot_description)/urdf/tripod.macro.xacro"/>
-    <xacro:include filename="$(find mmtbot_description)/urdf/astra.urdf.xacro" />
-<!--    <xacro:include filename="$(find ur_e_description)/urdf/common.gazebo.xacro" />-->
-<!--    <xacro:include filename="$(find ur_e_description)/urdf/ur10e.urdf.xacro" />-->
-    <xacro:include filename="$(find velodyne_description)/urdf/VLP-16.urdf.xacro"/>
-    <!-- Links and joints-->
-    <link name="world"/>
-    <!-- Place table 1 in the scene-->
-    <xacro:table_macro name="table" parent="world" width="${table_width}"
-                       lenght="${table_lenght}" height="${table_height}"
-                       tabletop_thickness="${table_tabletop_thickness}" leg_radius="${table_leg_radius}">
-        <origin xyz="-1 0 0" rpy="0 0 ${M_PI/2}" />
-    </xacro:table_macro>
-    <!--  Manipulator-->
-        <!--   UR10e properties -->
-    <!-- parameters -->
+    <!-- Manipulator's args and propperties -->
     <xacro:arg name="joint_limit_params" default=""/>
     <xacro:arg name="kinematics_params" default=""/>
@@ -44,15 +28,38 @@
     <xacro:arg name="safety_pos_margin" default="0.15"/>
     <xacro:arg name="safety_k_position" default="20"/>
-<!--    <xacro:ur10e_robot prefix="" joint_limited="false"/>-->
-    <xacro:include filename="$(find ur_description)/urdf/inc/ur10e_macro.xacro"/>
-    <xacro:ur10e_robot prefix=""
-        joint_limits_parameters_file="$(arg joint_limit_params)"
-        kinematics_parameters_file="$(arg kinematics_params)"
-        physical_parameters_file="$(arg physical_params)"
-        visual_parameters_file="$(arg visual_params)"
-        transmission_hw_interface="$(arg transmission_hw_interface)"
-        safety_limits="$(arg safety_limits)"
-        safety_pos_margin="$(arg safety_pos_margin)"
-        safety_k_position="$(arg safety_k_position)"
+    <!-- ####################################### -->
+    <!-- Include files-->
+    <!-- ####################################### -->
+    <!-- Scene objets-->
+    <xacro:include filename="$(find mmtbot_description)/urdf/properties.xacro"/>
+    <xacro:include filename="$(find mmtbot_description)/urdf/table.macro.xacro"/>
+    <xacro:include filename="$(find mmtbot_description)/urdf/tripod.macro.xacro"/>
+    <!-- Sensors-->
+    <xacro:include filename="$(find mmtbot_description)/urdf/astra.urdf.xacro" />
+    <xacro:include filename="$(find velodyne_description)/urdf/VLP-16.urdf.xacro"/>
+    <!-- Manipulator-->
+    <xacro:include filename="$(find ur_gazebo)/urdf/ur_macro.xacro"/>
+    <!--    <xacro:include filename="$(find ur_description)/urdf/inc/ur10e_macro.xacro"/>-->
+    <!-- ####################################### -->
+    <!-- Declare links and joints -->
+    <!-- ####################################### -->
+    <link name="world"/>
+    <!-- Place table 1 in the scene-->
+    <xacro:table_macro name="table" parent="world" width="${table_width}"
+                       lenght="${table_lenght}" height="${table_height}"
+                       tabletop_thickness="${table_tabletop_thickness}" leg_radius="${table_leg_radius}">
+        <origin xyz="-1 0 0" rpy="0 0 ${M_PI/2}" />
+    </xacro:table_macro>
+    <!--  Place manipulator1 in the scene-->
+    <xacro:ur_robot_gazebo
+            prefix=""
+            joint_limits_parameters_file="$(arg joint_limit_params)"
+            kinematics_parameters_file="$(arg kinematics_params)"
+            physical_parameters_file="$(arg physical_params)"
+            visual_parameters_file="$(arg visual_params)"
+            transmission_hw_interface="$(arg transmission_hw_interface)"
+            safety_limits="$(arg safety_limits)"
+            safety_pos_margin="$(arg safety_pos_margin)"
+            safety_k_position="$(arg safety_k_position)"
     />
     <!--  Place robot on top of the table1-->
@@ -62,7 +69,8 @@
         <origin xyz="0.0 0.0 0.001" rpy="0.0 0.0 0.0" />
     </joint>
-<!--    <xacro:sensor_astra prefix="hand_camera" parent="ee_link">-->
-<!--        <origin xyz="-0.02 0.05 0.07" rpy="0 0.0 0" />-->
-<!--    </xacro:sensor_astra>-->
+    <!-- Place hand camera 1 in the scene-->
+    <xacro:sensor_astra prefix="hand_camera" parent="flange">
+        <origin xyz="-0.02 0.05 0.07" rpy="0 0.0 0" />
+    </xacro:sensor_astra>
     <!-- Place tripod in the scene-->
     <xacro:tripod_macro name="tripod" parent="world">
