Commit message: Removing dependencies from Eurico's iris_ur10e packages

File: mmtbot_description/urdf/astra.urdf.xacro (robot description, xacro)
@@ -17,5 +17,5 @@
         <origin xyz="-0.03 -0.06 0" rpy="${pi} 0 ${pi/2}"/>
         <geometry>
-          <mesh filename="package://ur_e_description/meshes/sensors/astra2.dae" scale="1 1 1"/>
+          <mesh filename="package://mmtbot_description/meshes/astra2/astra2.dae" scale="1 1 1"/>
         </geometry>
       </visual>

File: mmtbot_description/urdf/mmtbot.urdf.xacro (robot description, xacro)
@@ -17,6 +17,6 @@
     <xacro:include filename="$(find mmtbot_description)/urdf/tripod.macro.xacro"/>
     <xacro:include filename="$(find mmtbot_description)/urdf/astra.urdf.xacro" />
-    <xacro:include filename="$(find ur_e_description)/urdf/common.gazebo.xacro" />
-    <xacro:include filename="$(find ur_e_description)/urdf/ur10e.urdf.xacro" />
+<!--    <xacro:include filename="$(find ur_e_description)/urdf/common.gazebo.xacro" />-->
+<!--    <xacro:include filename="$(find ur_e_description)/urdf/ur10e.urdf.xacro" />-->
     <xacro:include filename="$(find velodyne_description)/urdf/VLP-16.urdf.xacro"/>
     <!-- Links and joints-->
@@ -29,5 +29,31 @@
     </xacro:table_macro>
     <!--  Manipulator-->
-    <xacro:ur10e_robot prefix="" joint_limited="false"/>
+        <!--   UR10e properties -->
+    <!-- parameters -->
+    <xacro:arg name="joint_limit_params" default=""/>
+    <xacro:arg name="kinematics_params" default=""/>
+    <xacro:arg name="physical_params" default=""/>
+    <xacro:arg name="visual_params" default=""/>
+    <!-- legal values:
+          - hardware_interface/PositionJointInterface
+          - hardware_interface/VelocityJointInterface
+          - hardware_interface/EffortJointInterface
+    -->
+    <xacro:arg name="transmission_hw_interface" default="hardware_interface/PositionJointInterface"/>
+    <xacro:arg name="safety_limits" default="false"/>
+    <xacro:arg name="safety_pos_margin" default="0.15"/>
+    <xacro:arg name="safety_k_position" default="20"/>
+<!--    <xacro:ur10e_robot prefix="" joint_limited="false"/>-->
+    <xacro:include filename="$(find ur_description)/urdf/inc/ur10e_macro.xacro"/>
+    <xacro:ur10e_robot prefix=""
+        joint_limits_parameters_file="$(arg joint_limit_params)"
+        kinematics_parameters_file="$(arg kinematics_params)"
+        physical_parameters_file="$(arg physical_params)"
+        visual_parameters_file="$(arg visual_params)"
+        transmission_hw_interface="$(arg transmission_hw_interface)"
+        safety_limits="$(arg safety_limits)"
+        safety_pos_margin="$(arg safety_pos_margin)"
+        safety_k_position="$(arg safety_k_position)"
+    />
     <!--  Place robot on top of the table1-->
     <joint name="tabletop_table_to_ur10e" type="fixed">
@@ -36,7 +62,7 @@
         <origin xyz="0.0 0.0 0.001" rpy="0.0 0.0 0.0" />
     </joint>
-    <xacro:sensor_astra prefix="hand_camera" parent="ee_link">
-        <origin xyz="-0.02 0.05 0.07" rpy="0 0.0 0" />
-    </xacro:sensor_astra>
+<!--    <xacro:sensor_astra prefix="hand_camera" parent="ee_link">-->
+<!--        <origin xyz="-0.02 0.05 0.07" rpy="0 0.0 0" />-->
+<!--    </xacro:sensor_astra>-->
     <!-- Place tripod in the scene-->
     <xacro:tripod_macro name="tripod" parent="world">

Commit message: lardemua/atom#327 separating RGB and depth components

File: mmtbot_description/urdf/astra.urdf.xacro (robot description, xacro)
@@ -1,106 +1,144 @@
 <?xml version="1.0"?>
 <robot name="sensor_astra" xmlns:xacro="http://ros.org/wiki/xacro">
-  <!-- Xacro properties -->
-  <xacro:property name="astra_cam_py" value="-0.0125"/>
-  <xacro:property name="astra_depth_rel_rgb_py" value="0.0250" />
-  <xacro:property name="astra_cam_rel_rgb_py"   value="-0.0125" />
-  <xacro:property name="astra_dae_display_scale"   value="0.1" />
-  <!-- Parameterised in part by the values in turtlebot_properties.urdf.xacro -->
-  <xacro:macro name="sensor_astra" params="parent prefix *origin">
-    <joint name="${prefix}_joint" type="fixed">
-      <xacro:insert_block name="origin" />
-      <parent link="${parent}"/>
-      <child link="${prefix}_link"/>
-    </joint>
-    <link name="${prefix}_link">
-      <visual>
-        <origin xyz="-0.03 -0.06 0" rpy="${pi} 0 ${pi/2}"/>
-        <geometry>
-          <mesh filename="package://mmtbot_description/meshes/astra2/astra2.dae" scale="1 1 1"/>
-        </geometry>
-      </visual>
-      <collision>
-        <!-- <origin xyz="0.0 0.0 0.0" rpy="0 0 0" /> -->
-        <origin xyz="-0.01 -0.06 0" rpy="0 0 0"/>
-        <geometry>
-        <box size="0.0400 0.1650 0.0300"/>
-      </geometry>
-      </collision>
-      <inertial>
-        <mass value="0.564" />
-        <origin xyz="0 0 0" />
-        <inertia ixx="0.003881243" ixy="0.0" ixz="0.0"
-                 iyy="0.000498940" iyz="0.0"
-                 izz="0.003879257" />
-      </inertial>
-    </link>
-    <gazebo reference="${prefix}_link">
-      <selfCollide>false</selfCollide>
-    </gazebo>
-    <joint name="${prefix}_rgb_joint" type="fixed">
-      <origin xyz="0 -0.045 0" rpy="0 0 0" />
-      <parent link="${prefix}_link"/>
-      <child link="${prefix}_rgb_frame" />
-    </joint>
-    <link name="${prefix}_rgb_frame"/>
-    <joint name="${prefix}_rgb_optical_joint" type="fixed">
-      <origin xyz="0 0 0" rpy="${-pi/2} 0 ${-pi/2}" />
-      <parent link="${prefix}_rgb_frame" />
-      <child link="${prefix}_rgb_optical_frame" />
-    </joint>
-    <link name="${prefix}_rgb_optical_frame"/>
-    <joint name="${prefix}_depth_joint" type="fixed">
-        <origin xyz="0 -0.02 0" rpy="0 0 0" />
-        <parent link="${prefix}_link" />
-        <child link="${prefix}_depth_frame" />
-    </joint>
-    <link name="${prefix}_depth_frame"/>
-    <joint name="${prefix}_depth_optical_joint" type="fixed">
-        <origin xyz="0 0 0" rpy="${-pi/2} 0 ${-pi/2}" />
-        <parent link="${prefix}_depth_frame" />
-        <child link="${prefix}_depth_optical_frame" />
-    </joint>
-    <link name="${prefix}_depth_optical_frame"/>
-     <gazebo reference="${prefix}_depth_frame">
-          <sensor type="depth" name="camera">
-              <always_on>true</always_on>
-              <update_rate>10.0</update_rate>
-              <camera>
-                  <horizontal_fov>${60.0*pi/180.0}</horizontal_fov>
-                  <image>
-                      <format>B8G8R8</format>
-<!--                      <format>RGB_INT8</format>-->
-                      <width>1280</width>
-                      <height>720</height>
-                  </image>
-                  <clip>
-                      <near>0.10</near>
-                      <far>8.0</far>
-                  </clip>
-              </camera>
-              <plugin name="${prefix}_camera_controller" filename="libgazebo_ros_openni_kinect.so">
-                  <cameraName>${prefix}</cameraName>
-                  <alwaysOn>true</alwaysOn>
-                  <updateRate>0</updateRate>
-                  <imageTopicName>rgb/image_raw</imageTopicName>
-                  <depthImageTopicName>depth/image_raw</depthImageTopicName>
-                  <pointCloudTopicName>depth/points</pointCloudTopicName>
-                  <cameraInfoTopicName>rgb/camera_info</cameraInfoTopicName>
-                  <depthImageCameraInfoTopicName>depth/camera_info</depthImageCameraInfoTopicName>
-<!--                  <frameName>${prefix}_depth_optical_frame</frameName>-->
-<!--                  <frameName>${prefix}_rgb_optical_frame</frameName>-->
-                  <frameName>${prefix}_link</frameName>
-                  <!-- Apparently this is not used-->
-                  <baseline>0.1</baseline>
-<!--                  <hackBaseline>2</hackBaseline>-->
-                  <distortion_k1>0.0</distortion_k1>
-                  <distortion_k2>0.0</distortion_k2>
-                  <distortion_k3>0.0</distortion_k3>
-                  <distortion_t1>0.0</distortion_t1>
-                  <distortion_t2>0.0</distortion_t2>
-                  <pointCloudCutoff>0.4</pointCloudCutoff>
-              </plugin>
-          </sensor>
-      </gazebo>
-  </xacro:macro>
+    <!-- Xacro properties -->
+    <xacro:property name="astra_cam_py" value="-0.0125"/>
+    <xacro:property name="astra_depth_rel_rgb_py" value="0.0250"/>
+    <xacro:property name="astra_cam_rel_rgb_py" value="-0.0125"/>
+    <xacro:property name="astra_dae_display_scale" value="0.1"/>
+    <!-- Parameterised in part by the values in turtlebot_properties.urdf.xacro -->
+    <xacro:macro name="sensor_astra" params="parent prefix *origin">
+        <joint name="${prefix}_joint" type="fixed">
+            <xacro:insert_block name="origin"/>
+            <parent link="${parent}"/>
+            <child link="${prefix}_link"/>
+        </joint>
+        <link name="${prefix}_link">
+            <visual>
+                <origin xyz="-0.03 -0.06 0" rpy="${pi} 0 ${pi/2}"/>
+                <geometry>
+                    <mesh filename="package://mmtbot_description/meshes/astra2/astra2.dae" scale="1 1 1"/>
+                </geometry>
+            </visual>
+            <collision>
+                <!-- <origin xyz="0.0 0.0 0.0" rpy="0 0 0" /> -->
+                <origin xyz="-0.01 -0.06 0" rpy="0 0 0"/>
+                <geometry>
+                    <box size="0.0400 0.1650 0.0300"/>
+                </geometry>
+            </collision>
+            <inertial>
+                <mass value="0.564"/>
+                <origin xyz="0 0 0"/>
+                <inertia ixx="0.003881243" ixy="0.0" ixz="0.0"
+                         iyy="0.000498940" iyz="0.0"
+                         izz="0.003879257"/>
+            </inertial>
+        </link>
+        <gazebo reference="${prefix}_link">
+            <selfCollide>false</selfCollide>
+        </gazebo>
+        <joint name="${prefix}_rgb_joint" type="fixed">
+            <origin xyz="0 -0.045 0" rpy="0 0 0"/>
+            <parent link="${prefix}_link"/>
+            <child link="${prefix}_rgb_frame"/>
+        </joint>
+        <link name="${prefix}_rgb_frame"/>
+        <joint name="${prefix}_rgb_optical_joint" type="fixed">
+            <origin xyz="0 0 0" rpy="${-pi/2} 0 ${-pi/2}"/>
+            <parent link="${prefix}_rgb_frame"/>
+            <child link="${prefix}_rgb_optical_frame"/>
+        </joint>
+        <link name="${prefix}_rgb_optical_frame"/>
+        <joint name="${prefix}_depth_joint" type="fixed">
+            <origin xyz="0 -0.02 0" rpy="0 0 0"/>
+            <parent link="${prefix}_link"/>
+            <child link="${prefix}_depth_frame"/>
+        </joint>
+        <link name="${prefix}_depth_frame"/>
+        <joint name="${prefix}_depth_optical_joint" type="fixed">
+            <origin xyz="0 0 0" rpy="${-pi/2} 0 ${-pi/2}"/>
+            <parent link="${prefix}_depth_frame"/>
+            <child link="${prefix}_depth_optical_frame"/>
+        </joint>
+        <link name="${prefix}_depth_optical_frame"/>
+        <gazebo reference="${prefix}_link">
+            <sensor type="depth" name="camera">
+                <always_on>true</always_on>
+                <update_rate>10.0</update_rate>
+                <camera>
+                    <horizontal_fov>${60.0*pi/180.0}</horizontal_fov>
+                    <image>
+                        <format>B8G8R8</format>
+                        <!--                      <format>RGB_INT8</format>-->
+                        <width>1280</width>
+                        <height>720</height>
+                    </image>
+                    <clip>
+                        <near>0.10</near>
+                        <far>8.0</far>
+                    </clip>
+                </camera>
+                <plugin name="${prefix}_depth_camera_controller" filename="libgazebo_ros_openni_kinect.so">
+                    <cameraName>${prefix}</cameraName>
+                    <alwaysOn>true</alwaysOn>
+                    <updateRate>0</updateRate>
+                    <!--                  <imageTopicName>rgb/image_raw</imageTopicName>-->
+                    <depthImageTopicName>depth/image_raw</depthImageTopicName>
+                    <pointCloudTopicName>depth/points</pointCloudTopicName>
+                    <!--                  <cameraInfoTopicName>rgb/camera_info</cameraInfoTopicName>-->
+                    <depthImageCameraInfoTopicName>depth/camera_info</depthImageCameraInfoTopicName>
+                    <frameName>${prefix}_depth_optical_frame</frameName>
+                    <!--                  <frameName>${prefix}_rgb_optical_frame</frameName>-->
+                    <!--                  <frameName>${prefix}_link</frameName>-->
+                    <!-- Apparently this is not used-->
+                    <baseline>0.1</baseline>
+                    <!--                  <hackBaseline>2</hackBaseline>-->
+                    <distortion_k1>0.0</distortion_k1>
+                    <distortion_k2>0.0</distortion_k2>
+                    <distortion_k3>0.0</distortion_k3>
+                    <distortion_t1>0.0</distortion_t1>
+                    <distortion_t2>0.0</distortion_t2>
+                    <pointCloudCutoff>0.4</pointCloudCutoff>
+                </plugin>
+            </sensor>
+            <sensor type="camera" name="camera">
+                <update_rate>30.0</update_rate>
+                <camera>
+                    <horizontal_fov>${60.0*pi/180.0}</horizontal_fov>
+                    <image>
+                        <format>B8G8R8</format>
+                        <!--                      <format>RGB_INT8</format>-->
+                        <width>1280</width>
+                        <height>720</height>
+                    </image>
+                    <clip>
+                        <near>0.10</near>
+                        <far>8.0</far>
+                    </clip>
+                </camera>
+                <plugin name="${prefix}_rgb_camera_controller" filename="libgazebo_ros_camera.so">
+                    <cameraName>${prefix}</cameraName>
+                    <alwaysOn>true</alwaysOn>
+                    <updateRate>0</updateRate>
+                    <imageTopicName>rgb/image_raw</imageTopicName>
+                    <!--                    <depthImageTopicName>depth/image_raw</depthImageTopicName>-->
+                    <!--                    <pointCloudTopicName>depth/points</pointCloudTopicName>-->
+                    <cameraInfoTopicName>rgb/camera_info</cameraInfoTopicName>
+                    <!--                    <depthImageCameraInfoTopicName>depth/camera_info</depthImageCameraInfoTopicName>-->
+                    <!--                    <frameName>${prefix}_depth_optical_frame</frameName>-->
+                    <frameName>${prefix}_rgb_optical_frame</frameName>
+                    <!--                  <frameName>${prefix}_link</frameName>-->
+                    <!-- Apparently this is not used-->
+                    <baseline>0.1</baseline>
+                    <!--                  <hackBaseline>2</hackBaseline>-->
+                    <distortion_k1>0.0</distortion_k1>
+                    <distortion_k2>0.0</distortion_k2>
+                    <distortion_k3>0.0</distortion_k3>
+                    <distortion_t1>0.0</distortion_t1>
+                    <distortion_t2>0.0</distortion_t2>
+                    <pointCloudCutoff>0.4</pointCloudCutoff>
+                </plugin>
+            </sensor>
+        </gazebo>
+    </xacro:macro>
 </robot>

Commit message: lardemua/atom#327 correcting rgb_optical_frame

File: mmtbot_description/urdf/astra.urdf.xacro (robot description, xacro)
@@ -45,5 +45,6 @@
         <link name="${prefix}_rgb_frame"/>
         <joint name="${prefix}_rgb_optical_joint" type="fixed">
-            <origin xyz="0 0 0" rpy="${-pi/2} 0 ${-pi/2}"/>
+<!--            <origin xyz="0 0 0" rpy="${-pi/2} 0 ${-pi/2}"/>-->
+            <origin xyz="0 0 0" rpy="0 0 0"/>
             <parent link="${prefix}_rgb_frame"/>
             <child link="${prefix}_rgb_optical_frame"/>
@@ -62,5 +63,5 @@
         </joint>
         <link name="${prefix}_depth_optical_frame"/>
-        <gazebo reference="${prefix}_link">
+        <gazebo reference="${prefix}_depth_optical_frame">
             <sensor type="depth" name="camera">
                 <always_on>true</always_on>
@@ -102,7 +103,10 @@
                 </plugin>
             </sensor>
+        </gazebo>
+        <gazebo reference="${prefix}_rgb_optical_frame">
             <sensor type="camera" name="camera">
                 <update_rate>30.0</update_rate>
                 <camera>
+<!--                    <pose>0 0 0 ${M_PI/2} ${-M_PI/2} 0</pose>-->
                     <horizontal_fov>${60.0*pi/180.0}</horizontal_fov>
                     <image>
@@ -137,5 +141,5 @@
                     <distortion_t1>0.0</distortion_t1>
                     <distortion_t2>0.0</distortion_t2>
-                    <pointCloudCutoff>0.4</pointCloudCutoff>
+<!--                    <pointCloudCutoff>0.4</pointCloudCutoff>-->
                 </plugin>
             </sensor>

Commit message: #327 new version of astra xacro

File: mmtbot_description/urdf/astra.urdf.xacro (robot description, xacro)
@@ -45,6 +45,6 @@
         <link name="${prefix}_rgb_frame"/>
         <joint name="${prefix}_rgb_optical_joint" type="fixed">
-<!--            <origin xyz="0 0 0" rpy="${-pi/2} 0 ${-pi/2}"/>-->
-            <origin xyz="0 0 0" rpy="0 0 0"/>
+            <origin xyz="0 0 0" rpy="${-pi/2} 0 ${-pi/2}"/>
+<!--            <origin xyz="0 0 0" rpy="0 0 0"/>-->
             <parent link="${prefix}_rgb_frame"/>
             <child link="${prefix}_rgb_optical_frame"/>
@@ -63,5 +63,5 @@
         </joint>
         <link name="${prefix}_depth_optical_frame"/>
-        <gazebo reference="${prefix}_depth_optical_frame">
+        <gazebo reference="${prefix}_depth_frame">
             <sensor type="depth" name="camera">
                 <always_on>true</always_on>
@@ -83,6 +83,8 @@
                     <cameraName>${prefix}</cameraName>
                     <alwaysOn>true</alwaysOn>
-                    <updateRate>0</updateRate>
-                    <!--                  <imageTopicName>rgb/image_raw</imageTopicName>-->
+                    <updateRate>10.0</updateRate>
+<!--                                      <imageTopicName>rgb/image_raw</imageTopicName>-->
+                    <imageTopicName>null</imageTopicName>
+                    <cameraInfoTopicName>null/camera_info</cameraInfoTopicName>
                     <depthImageTopicName>depth/image_raw</depthImageTopicName>
                     <pointCloudTopicName>depth/points</pointCloudTopicName>
@@ -104,5 +106,5 @@
             </sensor>
         </gazebo>
-        <gazebo reference="${prefix}_rgb_optical_frame">
+        <gazebo reference="${prefix}_rgb_frame">
             <sensor type="camera" name="camera">
                 <update_rate>30.0</update_rate>

Commit message: lardemua/atom#345 creating visual shape for depth camera

File: mmtbot_description/urdf/astra.urdf.xacro (robot description, xacro)
@@ -46,5 +46,5 @@
         <joint name="${prefix}_rgb_optical_joint" type="fixed">
             <origin xyz="0 0 0" rpy="${-pi/2} 0 ${-pi/2}"/>
-<!--            <origin xyz="0 0 0" rpy="0 0 0"/>-->
+            <!--            <origin xyz="0 0 0" rpy="0 0 0"/>-->
             <parent link="${prefix}_rgb_frame"/>
             <child link="${prefix}_rgb_optical_frame"/>
@@ -62,5 +62,13 @@
             <child link="${prefix}_depth_optical_frame"/>
         </joint>
-        <link name="${prefix}_depth_optical_frame"/>
+        <link name="${prefix}_depth_optical_frame">
+            <visual>
+                <origin xyz="0 0 0.025" rpy="0 0 0"/>
+                <geometry>
+                    <cylinder length="0.05" radius="0.025"/>
+                </geometry>
+                <material name="Orange"></material>
+            </visual>
+        </link>
         <gazebo reference="${prefix}_depth_frame">
             <sensor type="depth" name="camera">
@@ -84,5 +92,5 @@
                     <alwaysOn>true</alwaysOn>
                     <updateRate>10.0</updateRate>
-<!--                                      <imageTopicName>rgb/image_raw</imageTopicName>-->
+                    <!--                                      <imageTopicName>rgb/image_raw</imageTopicName>-->
                     <imageTopicName>null</imageTopicName>
                     <cameraInfoTopicName>null/camera_info</cameraInfoTopicName>
@@ -110,5 +118,5 @@
                 <update_rate>30.0</update_rate>
                 <camera>
-<!--                    <pose>0 0 0 ${M_PI/2} ${-M_PI/2} 0</pose>-->
+                    <!--                    <pose>0 0 0 ${M_PI/2} ${-M_PI/2} 0</pose>-->
                     <horizontal_fov>${60.0*pi/180.0}</horizontal_fov>
                     <image>
@@ -143,5 +151,5 @@
                     <distortion_t1>0.0</distortion_t1>
                     <distortion_t2>0.0</distortion_t2>
-<!--                    <pointCloudCutoff>0.4</pointCloudCutoff>-->
+                    <!--                    <pointCloudCutoff>0.4</pointCloudCutoff>-->
                 </plugin>
             </sensor>
