Commit message: Setting up rviz pannel interaction with set_initial_estimate (#278)

File: mmtbot_calibration/urdf/initial_estimate.urdf.xacro (robot description, xacro)
@@ -1,52 +1,943 @@
 <?xml version="1.0" ?>
-<robot name="mmtbot" xmlns:xacro="http://ros.org/wiki/xacro">
-    <!--  Miguel Riem Oliveira-->
-    <!--  February 2021-->
-    <!--Args are local, properties are global, so we copy the values of the arguments to the properties-->
-    <!--Properties are global so they can be viewed from inside the included xacros-->
-    <!--  args are used with $(arg arg_name), properties are used as ${property_name}-->
-    <xacro:property name="table_height" value="0.795"/>
-    <xacro:property name="table_width" value=".9"/>
-    <xacro:property name="table_lenght" value="0.9"/>
-    <xacro:property name="table_tabletop_thickness" value="0.015"/>
-    <xacro:property name="table_leg_radius" value="0.02"/>
-    <xacro:property name="M_PI" value="3.1415926535897931" />
-    <!-- Include other files-->
-    <xacro:include filename="$(find mmtbot_description)/urdf/properties.xacro"/>
-    <xacro:include filename="$(find mmtbot_description)/urdf/table.macro.xacro"/>
-    <xacro:include filename="$(find mmtbot_description)/urdf/tripod.macro.xacro"/>
-    <xacro:include filename="$(find mmtbot_description)/urdf/astra.urdf.xacro" />
-    <xacro:include filename="$(find ur_e_description)/urdf/common.gazebo.xacro" />
-    <xacro:include filename="$(find ur_e_description)/urdf/ur10e.urdf.xacro" />
-    <xacro:include filename="$(find velodyne_description)/urdf/VLP-16.urdf.xacro"/>
-    <!-- Links and joints-->
-    <link name="world"/>
-    <!-- Place table 1 in the scene-->
-    <xacro:table_macro name="table" parent="world" width="${table_width}"
-                       lenght="${table_lenght}" height="${table_height}"
-                       tabletop_thickness="${table_tabletop_thickness}" leg_radius="${table_leg_radius}">
-        <origin xyz="-1 0 0" rpy="0 0 ${M_PI/2}" />
-    </xacro:table_macro>
-    <!--  Manipulator-->
-    <xacro:ur10e_robot prefix="" joint_limited="false"/>
-    <!--  Place robot on top of the table1-->
-    <joint name="tabletop_table_to_ur10e" type="fixed">
-        <parent link="tabletop_table" />
-        <child link = "base_link"/>
-        <origin xyz="0.0 0.0 0.001" rpy="0.0 0.0 0.0" />
+<robot name="mmtbot" version="1.0">
+  <material name="Yellow">
+    <color rgba="1.0 1.0 0.0 1.0"/>
+  </material>
+  <material name="Orange">
+    <color rgba="1.0 0.4 0.0 1.0"/>
+  </material>
+  <material name="grey">
+    <color rgba="0.7 0.7 0.7 1.0"/>
+  </material>
+  <gazebo>
+    <plugin filename="libgazebo_ros_control.so" name="ros_control">
+    </plugin>
+  </gazebo>
+  <link name="world"/>
+  <link name="table"/>
+  <joint name="world_to_table" type="fixed">
+    <origin xyz="-1.0 0.0 0.0" rpy="0.0 0.0 1.5707963267948966"/>
+    <parent link="world"/>
+    <child link="table"/>
+  </joint>
+  <link name="tabletop_table">
+    <inertial>
+      <origin xyz="0.0 0.0 -0.015" rpy="0.0 0.0 0.0"/>
+      <mass value="1.0"/>
+      <inertia ixx="1.0" ixy="0.0" ixz="0.0" iyy="1.0" iyz="0.0" izz="1.0"/>
+    </inertial>
+    <visual>
+      <origin xyz="0.0 0.0 -0.015" rpy="0.0 0.0 0.0"/>
+      <geometry>
+        <box size="0.9 0.9 0.015"/>
+      </geometry>
+      <material name="grey"/>
+    </visual>
+    <collision>
+      <origin xyz="0.0 0.0 -0.015" rpy="0.0 0.0 0.0"/>
+      <geometry>
+        <box size="0.9 0.9 0.015"/>
+      </geometry>
+    </collision>
+  </link>
+  <gazebo reference="tabletop_table">
+    <material>Gazebo/Grey</material>
+    <mu1>50.0</mu1>
+    <mu2>50.0</mu2>
+    <kp>1000000.0</kp>
+    <kd>1.0</kd>
+    <selfCollide>false</selfCollide>
+  </gazebo>
+  <joint name="table_to_tabletop_table" type="fixed">
+    <origin xyz="0.0 0.0 0.795" rpy="0.0 0.0 0.0"/>
+    <parent link="table"/>
+    <child link="tabletop_table"/>
+  </joint>
+  <link name="leg1_table">
+    <inertial>
+      <origin xyz="0.0 0.0 0.3815" rpy="0.0 0.0 0.0"/>
+      <mass value="1.0"/>
+      <inertia ixx="0.1" ixy="0.0" ixz="0.0" iyy="0.1" iyz="0.0" izz="0.01"/>
+    </inertial>
+    <visual>
+      <origin xyz="0.0 0.0 0.3815" rpy="0.0 0.0 0.0"/>
+      <geometry>
+        <cylinder radius="0.02" length="0.78"/>
+      </geometry>
+      <material name="grey"/>
+    </visual>
+    <collision>
+      <origin xyz="0.0 0.0 0.3975" rpy="0.0 0.0 0.0"/>
+      <geometry>
+        <cylinder radius="0.02" length="0.779"/>
+      </geometry>
+    </collision>
+  </link>
+  <gazebo reference="leg1_table">
+    <material>Gazebo/Grey</material>
+    <mu1>1000.0</mu1>
+    <mu2>1000.0</mu2>
+    <kp>10000000.0</kp>
+    <kd>1.0</kd>
+    <selfCollide>true</selfCollide>
+  </gazebo>
+  <joint name="table_to_leg1" type="fixed">
+    <origin xyz="-0.43 0.43 0.0" rpy="0.0 0.0 0.0"/>
+    <parent link="table"/>
+    <child link="leg1_table"/>
+  </joint>
+  <link name="leg2_table">
+    <inertial>
+      <origin xyz="0.0 0.0 0.3815" rpy="0.0 0.0 0.0"/>
+      <mass value="1.0"/>
+      <inertia ixx="0.1" ixy="0.0" ixz="0.0" iyy="0.1" iyz="0.0" izz="0.01"/>
+    </inertial>
+    <visual>
+      <origin xyz="0.0 0.0 0.3815" rpy="0.0 0.0 0.0"/>
+      <geometry>
+        <cylinder radius="0.02" length="0.78"/>
+      </geometry>
+      <material name="grey"/>
+    </visual>
+    <collision>
+      <origin xyz="0.0 0.0 0.3975" rpy="0.0 0.0 0.0"/>
+      <geometry>
+        <cylinder radius="0.02" length="0.779"/>
+      </geometry>
+    </collision>
+  </link>
+  <gazebo reference="leg2_table">
+    <material>Gazebo/Grey</material>
+    <mu1>1000.0</mu1>
+    <mu2>1000.0</mu2>
+    <kp>10000000.0</kp>
+    <kd>1.0</kd>
+    <selfCollide>true</selfCollide>
+  </gazebo>
+  <joint name="table_to_leg2" type="fixed">
+    <origin xyz="0.43 0.43 0.0" rpy="0.0 0.0 0.0"/>
+    <parent link="table"/>
+    <child link="leg2_table"/>
+  </joint>
+  <link name="leg3_table">
+    <inertial>
+      <origin xyz="0.0 0.0 0.3815" rpy="0.0 0.0 0.0"/>
+      <mass value="1.0"/>
+      <inertia ixx="0.1" ixy="0.0" ixz="0.0" iyy="0.1" iyz="0.0" izz="0.01"/>
+    </inertial>
+    <visual>
+      <origin xyz="0.0 0.0 0.3815" rpy="0.0 0.0 0.0"/>
+      <geometry>
+        <cylinder radius="0.02" length="0.78"/>
+      </geometry>
+      <material name="grey"/>
+    </visual>
+    <collision>
+      <origin xyz="0.0 0.0 0.3975" rpy="0.0 0.0 0.0"/>
+      <geometry>
+        <cylinder radius="0.02" length="0.779"/>
+      </geometry>
+    </collision>
+  </link>
+  <gazebo reference="leg3_table">
+    <material>Gazebo/Grey</material>
+    <mu1>1000.0</mu1>
+    <mu2>1000.0</mu2>
+    <kp>10000000.0</kp>
+    <kd>1.0</kd>
+    <selfCollide>true</selfCollide>
+  </gazebo>
+  <joint name="table_to_leg3" type="fixed">
+    <origin xyz="0.43 -0.43 0.0" rpy="0.0 0.0 0.0"/>
+    <parent link="table"/>
+    <child link="leg3_table"/>
+  </joint>
+  <link name="leg4_table">
+    <inertial>
+      <origin xyz="0.0 0.0 0.3815" rpy="0.0 0.0 0.0"/>
+      <mass value="1.0"/>
+      <inertia ixx="0.1" ixy="0.0" ixz="0.0" iyy="0.1" iyz="0.0" izz="0.01"/>
+    </inertial>
+    <visual>
+      <origin xyz="0.0 0.0 0.3815" rpy="0.0 0.0 0.0"/>
+      <geometry>
+        <cylinder radius="0.02" length="0.78"/>
+      </geometry>
+      <material name="grey"/>
+    </visual>
+    <collision>
+      <origin xyz="0.0 0.0 0.3975" rpy="0.0 0.0 0.0"/>
+      <geometry>
+        <cylinder radius="0.02" length="0.779"/>
+      </geometry>
+    </collision>
+  </link>
+  <gazebo reference="leg4_table">
+    <material>Gazebo/Grey</material>
+    <mu1>1000.0</mu1>
+    <mu2>1000.0</mu2>
+    <kp>10000000.0</kp>
+    <kd>1.0</kd>
+    <selfCollide>true</selfCollide>
+  </gazebo>
+  <joint name="table_to_leg4" type="fixed">
+    <origin xyz="-0.43 -0.43 0.0" rpy="0.0 0.0 0.0"/>
+    <parent link="table"/>
+    <child link="leg4_table"/>
+  </joint>
+  <link name="base_link">
+    <inertial>
+      <origin xyz="0.0 0.0 0.0" rpy="0.0 0.0 0.0"/>
+      <mass value="4.0"/>
+      <inertia ixx="0.0061063308908" ixy="0.0" ixz="0.0" iyy="0.0061063308908" iyz="0.0" izz="0.01125"/>
+    </inertial>
+    <visual>
+      <geometry>
+        <mesh filename="package://ur_e_description/meshes/ur10e/visual/base.dae"/>
+      </geometry>
+      <material name="LightGrey">
+        <color rgba="0.7 0.7 0.7 1.0"/>
+      </material>
+    </visual>
+    <collision>
+      <geometry>
+        <mesh filename="package://ur_e_description/meshes/ur10e/collision/base.stl"/>
+      </geometry>
+    </collision>
+  </link>
+  <joint name="shoulder_pan_joint" type="revolute">
+    <origin xyz="0.0 0.0 0.1807183549475882" rpy="0.0 0.0 0.0"/>
+    <axis xyz="0.0 0.0 1.0"/>
+    <parent link="base_link"/>
+    <child link="shoulder_link"/>
+    <limit effort="330.0" lower="-6.283185307179586" upper="6.283185307179586" velocity="3.14"/>
+    <dynamics damping="0.0" friction="0.0"/>
+  </joint>
+  <link name="shoulder_link">
+    <inertial>
+      <origin xyz="0.0 0.0 0.0" rpy="0.0 0.0 0.0"/>
+      <mass value="7.369"/>
+      <inertia ixx="0.029819260655624295" ixy="0.0" ixz="0.0" iyy="0.029819260655624295" iyz="0.0" izz="0.020725312499999995"/>
+    </inertial>
+    <visual>
+      <geometry>
+        <mesh filename="package://ur_e_description/meshes/ur10e/visual/shoulder.dae"/>
+      </geometry>
+      <material name="LightGrey">
+        <color rgba="0.7 0.7 0.7 1.0"/>
+      </material>
+    </visual>
+    <collision>
+      <geometry>
+        <mesh filename="package://ur_e_description/meshes/ur10e/collision/shoulder.stl"/>
+      </geometry>
+    </collision>
+  </link>
+  <joint name="shoulder_lift_joint" type="revolute">
+    <origin xyz="0.0 0.176 0.0" rpy="0.0 1.5707963267948966 0.0"/>
+    <axis xyz="0.0 1.0 0.0"/>
+    <parent link="shoulder_link"/>
+    <child link="upper_arm_link"/>
+    <limit effort="330.0" lower="-6.283185307179586" upper="6.283185307179586" velocity="3.14"/>
+    <dynamics damping="0.0" friction="0.0"/>
+  </joint>
+  <link name="upper_arm_link">
+    <inertial>
+      <origin xyz="0.0 0.0 0.306104723041748" rpy="0.0 0.0 0.0"/>
+      <mass value="13.051"/>
+      <inertia ixx="0.4259794731131226" ixy="0.0" ixz="0.0" iyy="0.4259794731131226" iyz="0.0" izz="0.036705937499999994"/>
+    </inertial>
+    <visual>
+      <geometry>
+        <mesh filename="package://ur_e_description/meshes/ur10e/visual/upperarm.dae"/>
+      </geometry>
+      <material name="LightGrey">
+        <color rgba="0.7 0.7 0.7 1.0"/>
+      </material>
+    </visual>
+    <collision>
+      <geometry>
+        <mesh filename="package://ur_e_description/meshes/ur10e/collision/upperarm.stl"/>
+      </geometry>
+    </collision>
+  </link>
+  <joint name="elbow_joint" type="revolute">
+    <origin xyz="0.0 -0.137 0.612209446083496" rpy="0.0 0.0 0.0"/>
+    <axis xyz="0.0 1.0 0.0"/>
+    <parent link="upper_arm_link"/>
+    <child link="forearm_link"/>
+    <limit effort="150.0" lower="-3.141592653589793" upper="3.141592653589793" velocity="3.14"/>
+    <dynamics damping="0.0" friction="0.0"/>
+  </joint>
+  <link name="forearm_link">
+    <inertial>
+      <origin xyz="0.0 0.0 0.28550853623327865" rpy="0.0 0.0 0.0"/>
+      <mass value="3.989"/>
+      <inertia ixx="0.11399742921147499" ixy="0.0" ixz="0.0" iyy="0.11399742921147499" iyz="0.0" izz="0.011219062499999998"/>
+    </inertial>
+    <visual>
+      <geometry>
+        <mesh filename="package://ur_e_description/meshes/ur10e/visual/forearm.dae"/>
+      </geometry>
+      <material name="LightGrey">
+        <color rgba="0.7 0.7 0.7 1.0"/>
+      </material>
+    </visual>
+    <collision>
+      <geometry>
+        <mesh filename="package://ur_e_description/meshes/ur10e/collision/forearm.stl"/>
+      </geometry>
+    </collision>
+  </link>
+  <joint name="wrist_1_joint" type="revolute">
+    <origin xyz="0.0 0.0 0.5710170724665573" rpy="0.0 1.5707963267948966 0.0"/>
+    <axis xyz="0.0 1.0 0.0"/>
+    <parent link="forearm_link"/>
+    <child link="wrist_1_link"/>
+    <limit effort="54.0" lower="-6.283185307179586" upper="6.283185307179586" velocity="6.28"/>
+    <dynamics damping="0.0" friction="0.0"/>
+  </joint>
+  <link name="wrist_1_link">
+    <inertial>
+      <origin xyz="0.0 0.1347892222434263 0.0" rpy="0.0 0.0 0.0"/>
+      <mass value="2.1"/>
+      <inertia ixx="0.00547312281075" ixy="0.0" ixz="0.0" iyy="0.00547312281075" iyz="0.0" izz="0.00590625"/>
+    </inertial>
+    <visual>
+      <geometry>
+        <mesh filename="package://ur_e_description/meshes/ur10e/visual/wrist1.dae"/>
+      </geometry>
+      <material name="LightGrey">
+        <color rgba="0.7 0.7 0.7 1.0"/>
+      </material>
+    </visual>
+    <collision>
+      <geometry>
+        <mesh filename="package://ur_e_description/meshes/ur10e/collision/wrist1.stl"/>
+      </geometry>
+    </collision>
+  </link>
+  <joint name="wrist_2_joint" type="revolute">
+    <origin xyz="0.0 0.1347892222434263 0.0" rpy="0.0 0.0 0.0"/>
+    <axis xyz="0.0 0.0 1.0"/>
+    <parent link="wrist_1_link"/>
+    <child link="wrist_2_link"/>
+    <limit effort="54.0" lower="-6.283185307179586" upper="6.283185307179586" velocity="6.28"/>
+    <dynamics damping="0.0" friction="0.0"/>
+  </joint>
+  <link name="wrist_2_link">
+    <inertial>
+      <origin xyz="0.0 0.0 0.1198680944284703" rpy="0.0 0.0 0.0"/>
+      <mass value="1.98"/>
+      <inertia ixx="0.005160372935849999" ixy="0.0" ixz="0.0" iyy="0.005160372935849999" iyz="0.0" izz="0.00556875"/>
+    </inertial>
+    <visual>
+      <geometry>
+        <mesh filename="package://ur_e_description/meshes/ur10e/visual/wrist2.dae"/>
+      </geometry>
+      <material name="LightGrey">
+        <color rgba="0.7 0.7 0.7 1.0"/>
+      </material>
+    </visual>
+    <collision>
+      <geometry>
+        <mesh filename="package://ur_e_description/meshes/ur10e/collision/wrist2.stl"/>
+      </geometry>
+    </collision>
+  </link>
+  <joint name="wrist_3_joint" type="revolute">
+    <origin xyz="0.0 0.0 0.1198680944284703" rpy="0.0 0.0 0.0"/>
+    <axis xyz="0.0 1.0 0.0"/>
+    <parent link="wrist_2_link"/>
+    <child link="wrist_3_link"/>
+    <limit effort="54.0" lower="-6.283185307179586" upper="6.283185307179586" velocity="6.28"/>
+    <dynamics damping="0.0" friction="0.0"/>
+  </joint>
+  <link name="wrist_3_link">
+    <inertial>
+      <origin xyz="0.0 0.0906473542891715 0.0" rpy="1.5707963267948966 0.0 0.0"/>
+      <mass value="0.615"/>
+      <inertia ixx="0.0004394685742125001" ixy="0.0" ixz="0.0" iyy="0.0004394685742125001" iyz="0.0" izz="0.0006226875"/>
+    </inertial>
+    <visual>
+      <geometry>
+        <mesh filename="package://ur_e_description/meshes/ur10e/visual/wrist3.dae"/>
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
Commit message: #284 implemented from the set_initial_estimate side.

File: mmtbot_calibration/urdf/initial_estimate.urdf.xacro (robot description, xacro)
@@ -595,5 +595,5 @@
   </joint>
   <joint name="hand_camera_joint" type="fixed">
-    <origin xyz="-0.02 0.05 0.07" rpy="0.0 -0.0 0.0"/>
+    <origin xyz="0.7800358533859253 0.05000000074505806 0.07000000029802322" rpy="0.0 -0.0 0.0"/>
     <parent link="ee_link"/>
     <child link="hand_camera_link"/>
@@ -601,5 +601,5 @@
   <link name="hand_camera_link">
     <inertial>
-      <origin xyz="0.0 0.0 0.0" rpy="0 0 0"/>
+      <origin xyz="0.0 0.0 0.0" rpy="0.0 0.0 0.0"/>
       <mass value="0.564"/>
       <inertia ixx="0.003881243" ixy="0.0" ixz="0.0" iyy="0.00049894" iyz="0.0" izz="0.003879257"/>
@@ -768,5 +768,5 @@
   </joint>
   <joint name="3dlidar_base_mount_joint" type="fixed">
-    <origin xyz="0.0 0.0 0.001" rpy="0.0 -0.0 0.0"/>
+    <origin xyz="-0.8649045825004578 0.0 0.9622363448143005" rpy="0.0 -0.0 0.0"/>
     <parent link="tripod_left_support"/>
     <child link="3dlidar_base_link"/>
@@ -774,5 +774,5 @@
   <link name="3dlidar_base_link">
     <inertial>
-      <origin xyz="0.0 0.0 0.03585" rpy="0 0 0"/>
+      <origin xyz="0.0 0.0 0.03585" rpy="0.0 0.0 0.0"/>
       <mass value="0.83"/>
       <inertia ixx="0.000908059425" ixy="0.0" ixz="0.0" iyy="0.000908059425" iyz="0.0" izz="0.0011049624"/>
@@ -802,10 +802,10 @@
   <link name="3dlidar">
     <inertial>
-      <origin xyz="0.0 0.0 0.0" rpy="0 0 0"/>
+      <origin xyz="0.0 0.0 0.0" rpy="0.0 0.0 0.0"/>
       <mass value="0.01"/>
       <inertia ixx="1e-07" ixy="0.0" ixz="0.0" iyy="1e-07" iyz="0.0" izz="1e-07"/>
     </inertial>
     <visual>
-      <origin xyz="0.0 0.0 -0.0377" rpy="0 0 0"/>
+      <origin xyz="0.0 0.0 -0.0377" rpy="0.0 0.0 0.0"/>
       <geometry>
         <mesh filename="package://velodyne_description/meshes/VLP16_scan.dae"/>
@@ -855,5 +855,5 @@
   </gazebo>
   <joint name="world_camera_joint" type="fixed">
-    <origin xyz="0.02 0.07 0.015" rpy="0.0 -0.0 0.0"/>
+    <origin xyz="-1.0961196422576904 -1.1593269109725952 0.014999999664723873" rpy="-0.7709805919192392 0.2310411274833507 0.23146684024077507"/>
     <parent link="tripod_right_support"/>
     <child link="world_camera_link"/>
@@ -861,5 +861,5 @@
   <link name="world_camera_link">
     <inertial>
-      <origin xyz="0.0 0.0 0.0" rpy="0 0 0"/>
+      <origin xyz="0.0 0.0 0.0" rpy="0.0 0.0 0.0"/>
       <mass value="0.564"/>
       <inertia ixx="0.003881243" ixy="0.0" ixz="0.0" iyy="0.00049894" iyz="0.0" izz="0.003879257"/>
